File: PCB/EAGLE/BOTTOM/Bottom.sch (EAGLE design)
At the start: 81 parts, among them J1 \, J2 Anodes, J3 2X6 FEMALE, Q1 MMBTA42, Q10 MMBTA92, Q11 32.768, Q2 MMBTA42, Q3 MMBTA42, Q4 MMBTA42, Q5 MMBTA42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

Commit message: Update boards to latest, update packaging photos, add 3D printed part files
Parts:
- removed Q11: 32.768, microbuilder:CRYSTAL8.0X3.8
- C11, C12: value 22p -> 14pF
- U1: value DS1307 -> DS3231M; device microbuilder:RTC_DS1307 -> SparkFun-Clocks:DS3231M
Connections:
- removed net XI: Q11.1, U1.X1
- removed net XO: Q11.2, U1.X2
- net SQW: now also U1.SQW; no longer U1.SQW/OUT
Changed lines of the file:
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@@
 <part name="GND2" library="supply1" library_urn="urn:adsk.eagle:library:371" deviceset="GND" device=""/>
 <part name="GND3" library="supply1" library_urn="urn:adsk.eagle:library:371" deviceset="GND" device=""/>
-<part name="Q11" library="microbuilder" deviceset="CRYSTAL" device="8.0X3.8" value="32.768"/>
 <part name="GND17" library="supply1" library_urn="urn:adsk.eagle:library:371" deviceset="GND" device=""/>
-<part name="U1" library="microbuilder" deviceset="RTC_DS1307" device="" value="DS1307"/>
 <part name="GND5" library="supply1" library_urn="urn:adsk.eagle:library:371" deviceset="GND" device=""/>
 <part name="SUPPLY2" library="SparkFun-PowerSymbols" library_urn="urn:adsk.eagle:library:530" deviceset="VCC_2" device="" value="170V"/>
@@
 <part name="C9" library="SparkFun-Capacitors" library_urn="urn:adsk.eagle:library:510" deviceset="2.2UF" device="-0805-25V-(+80/-20%)" package3d_urn="urn:adsk.eagle:package:37429/1" value="1u"/>
 <part name="C10" library="SparkFun-Capacitors" library_urn="urn:adsk.eagle:library:510" deviceset="2.2UF" device="-0805-25V-(+80/-20%)" package3d_urn="urn:adsk.eagle:package:37429/1" value="100n"/>
-<part name="C11" library="SparkFun-Capacitors" library_urn="urn:adsk.eagle:library:510" deviceset="2.2UF" device="-0805-25V-(+80/-20%)" package3d_urn="urn:adsk.eagle:package:37429/1" value="22p"/>
-<part name="C12" library="SparkFun-Capacitors" library_urn="urn:adsk.eagle:library:510" deviceset="2.2UF" device="-0805-25V-(+80/-20%)" package3d_urn="urn:adsk.eagle:package:37429/1" value="22p"/>
+<part name="C11" library="SparkFun-Capacitors" library_urn="urn:adsk.eagle:library:510" deviceset="2.2UF" device="-0805-25V-(+80/-20%)" package3d_urn="urn:adsk.eagle:package:37429/1" value="14pF"/>
+<part name="C12" library="SparkFun-Capacitors" library_urn="urn:adsk.eagle:library:510" deviceset="2.2UF" device="-0805-25V-(+80/-20%)" package3d_urn="urn:adsk.eagle:package:37429/1" value="14pF"/>
 <part name="U3" library="SmartPrj" deviceset="ATMEGA32U4-XU" device="AU"/>
 <part name="P+8" library="supply1" library_urn="urn:adsk.eagle:library:371" deviceset="+5V" device=""/>
@@
 <part name="D1" library="MF_LEDs" deviceset="LED_SINGLE" device="-0805" value="red"/>
 <part name="C5" library="SparkFun-Capacitors" library_urn="urn:adsk.eagle:library:510" deviceset="2.2UF" device="-0805-25V-(+80/-20%)" package3d_urn="urn:adsk.eagle:package:37429/1" value="100n"/>
+<part name="U1" library="SparkFun-Clocks" library_urn="urn:adsk.eagle:library:511" deviceset="DS3231M" device="" package3d_urn="urn:adsk.eagle:package:37530/1"/>
 </parts>
 <sheets>
@@
 <attribute name="VALUE" x="33.02" y="76.2" size="1.778" layer="96"/>
 </instance>
-<instance part="Q11" gate="G$1" x="353.06" y="66.04" smashed="yes" rot="MR270">
-<attribute name="NAME" x="350.52" y="68.58" size="1.27" layer="95" rot="MR270"/>
-<attribute name="VALUE" x="356.87" y="68.58" size="1.27" layer="96" rot="MR270"/>
-</instance>
 <instance part="GND17" gate="1" x="347.98" y="43.18" smashed="yes">
 <attribute name="VALUE" x="345.44" y="40.64" size="1.778" layer="96"/>
-</instance>
-<instance part="U1" gate="G$1" x="378.46" y="78.74" smashed="yes" rot="MR0">
-<attribute name="NAME" x="388.62" y="99.06" size="1.27" layer="95" rot="MR0"/>
-<attribute name="VALUE" x="388.62" y="55.88" size="1.27" layer="96" rot="MR0"/>
 </instance>
 <instance part="GND5" gate="1" x="393.7" y="71.12" smashed="yes">
@@
 </instance>
 <instance part="R21" gate="G$1" x="205.74" y="160.02" smashed="yes" rot="R270">
-<attribute name="NAME" x="207.264" y="160.02" size="1.778" layer="95" font="vector" rot="R270" align="bottom-center"/>
-<attribute name="VALUE" x="204.216" y="160.02" size="1.778" layer="96" font="vector" rot="R270" align="top-center"/>
+<attribute name="NAME" x="207.01" y="160.782" size="1.778" layer="95" font="vector" rot="R270" align="bottom-center"/>
+<attribute name="VALUE" x="208.534" y="155.702" size="1.778" layer="96" font="vector" rot="R270" align="top-center"/>
 </instance>
 <instance part="R22" gate="G$1" x="213.36" y="162.56" smashed="yes" rot="R270">
-<attribute name="NAME" x="214.884" y="162.56" size="1.778" layer="95" font="vector" rot="R270" align="bottom-center"/>
+<attribute name="NAME" x="210.566" y="167.64" size="1.778" layer="95" font="vector" rot="R270" align="bottom-center"/>
 <attribute name="VALUE" x="211.836" y="162.56" size="1.778" layer="96" font="vector" rot="R270" align="top-center"/>
 </instance>
@@
 <instance part="R33" gate="G$1" x="218.44" y="162.56" smashed="yes" rot="R270">
 <attribute name="NAME" x="219.964" y="162.56" size="1.778" layer="95" font="vector" rot="R270" align="bottom-center"/>
-<attribute name="VALUE" x="216.916" y="162.56" size="1.778" layer="96" font="vector" rot="R270" align="top-center"/>
+<attribute name="VALUE" x="221.488" y="168.402" size="1.778" layer="96" font="vector" rot="R270" align="top-center"/>
 </instance>
 <instance part="R34" gate="G$1" x="200.66" y="160.02" smashed="yes" rot="R270">
-<attribute name="NAME" x="202.184" y="160.02" size="1.778" layer="95" font="vector" rot="R270" align="bottom-center"/>
-<attribute name="VALUE" x="199.136" y="160.02" size="1.778" layer="96" font="vector" rot="R270" align="top-center"/>
+<attribute name="NAME" x="197.104" y="162.56" size="1.778" layer="95" font="vector" rot="R270" align="bottom-center"/>
+<attribute name="VALUE" x="199.136" y="157.48" size="1.778" layer="96" font="vector" rot="R270" align="top-center"/>
 </instance>
 <instance part="FID1" gate="G$1" x="276.86" y="127" smashed="yes">
@@
 <attribute name="NAME" x="336.804" y="89.281" size="1.778" layer="95" font="vector"/>
 <attribute name="VALUE" x="336.804" y="84.201" size="1.778" layer="96" font="vector"/>
+</instance>
+<instance part="U1" gate="G$1" x="381" y="78.74" smashed="yes">
+<attribute name="NAME" x="373.38" y="87.122" size="1.778" layer="95" font="vector" ratio="10"/>
+<attribute name="VALUE" x="373.38" y="71.12" size="1.778" layer="96" font="vector" ratio="10"/>
 </instance>
 </instances>
@@
 </segment>
 <segment>
+<pinref part="GND5" gate="1" pin="GND"/>
+<wire x1="393.7" y1="73.66" x2="393.7" y2="76.2" width="0.1524" layer="91"/>
 <pinref part="U1" gate="G$1" pin="GND"/>
-<pinref part="GND5" gate="1" pin="GND"/>
-<wire x1="393.7" y1="73.66" x2="391.16" y2="73.66" width="0.1524" layer="91"/>
 </segment>
 <segment>
@@
 </segment>
 <segment>
+<wire x1="368.3" y1="81.28" x2="363.22" y2="81.28" width="0.1524" layer="91"/>
+<wire x1="363.22" y1="81.28" x2="363.22" y2="88.9" width="0.1524" layer="91"/>
+<pinref part="P+8" gate="1" pin="+5V"/>
 <pinref part="U1" gate="G$1" pin="VCC"/>
-<wire x1="365.76" y1="86.36" x2="363.22" y2="86.36" width="0.1524" layer="91"/>
-<wire x1="363.22" y1="86.36" x2="363.22" y2="88.9" width="0.1524" layer="91"/>
-<pinref part="P+8" gate="1" pin="+5V"/>
 </segment>
 <segment>
@@
 <net name="SDA" class="0">
 <segment>
+<wire x1="401.32" y1="81.28" x2="393.7" y2="81.28" width="0.1524" layer="91"/>
+<label x="396.24" y="81.28" size="1.778" layer="95"/>
 <pinref part="U1" gate="G$1" pin="SDA"/>
-<wire x1="365.76" y1="73.66" x2="353.06" y2="73.66" width="0.1524" layer="91"/>
-<label x="355.6" y="73.66" size="1.778" layer="95"/>
 </segment>
 <segment>
@@
 <net name="SCL" class="0">
 <segment>
+<wire x1="393.7" y1="83.82" x2="401.32" y2="83.82" width="0.1524" layer="91"/>
+<label x="396.24" y="83.82" size="1.778" layer="95"/>
 <pinref part="U1" gate="G$1" pin="SCL"/>
-<wire x1="353.06" y1="76.2" x2="365.76" y2="76.2" width="0.1524" layer="91"/>
-<label x="355.6" y="76.2" size="1.778" layer="95"/>
 </segment>
 <segment>
@@
 </segment>
 <segment>
+<wire x1="393.7" y1="78.74" x2="401.32" y2="78.74" width="0.1524" layer="91"/>
+<label x="396.24" y="78.74" size="1.778" layer="95"/>
 <pinref part="U1" gate="G$1" pin="VBAT"/>
-<wire x1="391.16" y1="76.2" x2="398.78" y2="76.2" width="0.1524" layer="91"/>
-<label x="393.7" y="76.2" size="1.778" layer="95"/>
 </segment>
 </net>
 <net name="SQW" class="0">
 <segment>
-<pinref part="U1" gate="G$1" pin="SQW/OUT"/>
-<wire x1="365.76" y1="81.28" x2="353.06" y2="81.28" width="0.1524" layer="91"/>
-<label x="355.6" y="81.28" size="1.778" layer="95"/>
-</segment>
-</net>
-<net name="XI" class="0">
-<segment>
-<pinref part="U1" gate="G$1" pin="X1"/>
-<wire x1="391.16" y1="86.36" x2="398.78" y2="86.36" width="0.1524" layer="91"/>
-<label x="393.7" y="86.36" size="1.778" layer="95"/>
-</segment>
-<segment>
-<pinref part="Q11" gate="G$1" pin="1"/>
-<wire x1="353.06" y1="68.58" x2="337.82" y2="68.58" width="0.1524" layer="91"/>
-<label x="337.82" y="68.58" size="1.778" layer="95"/>
-</segment>
-</net>
-<net name="XO" class="0">
-<segment>
-<pinref part="U1" gate="G$1" pin="X2"/>
-<wire x1="398.78" y1="81.28" x2="391.16" y2="81.28" width="0.1524" layer="91"/>
-<label x="393.7" y="81.28" size="1.778" layer="95"/>
-</segment>
-<segment>
-<wire x1="353.06" y1="63.5" x2="337.82" y2="63.5" width="0.1524" layer="91"/>
-<pinref part="Q11" gate="G$1" pin="2"/>
-<label x="337.82" y="63.5" size="1.778" layer="95"/>
-</segment>
-</net>
+<wire x1="368.3" y1="78.74" x2="360.68" y2="78.74" width="0.1524" layer="91"/>
+<label x="360.68" y="78.74" size="1.778" layer="95"/>
+<pinref part="U1" gate="G$1" pin="SQW"/>
+</segment>
+</net>
